File: KICAD/4mb mapper nms8280.kicad_sch (KiCad schematic)
At the start: 22 parts, among them IC131 74LS125, IC131B1 74LS125, IC131C1 74LS125, IC147 74LS157, IC147B1 74LS157, IC149 74LS670, IC149B1 74LS670, IC157B1 74LS08, IC180B1 74LS00, J1 Conn_01x10_Pin

Commit message: Publish 4 MB mapper project
Parts:
- IC149, IC149B1: footprint Package_SO:SOIC-16_3.9x9.9mm_P1.27mm -> Package_DIP:DIP-16_W7.62mm
Changed lines of the file:
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@@
-	(global_label "Vcc"
-		(shape input)
-		(at 267.97 59.69 0)
-		(fields_autoplaced yes)
-		(effects
-			(font
-				(size 0.762 0.762)
-			)
-			(justify left)
-		)
-		(property "Intersheetrefs" "${INTERSHEET_REFS}"
-			(at 271.7207 59.69 0)
-			(hide yes)
-			(show_name no)
-			(do_not_autoplace no)
-			(effects
-				(font
-					(size 1.27 1.27)
-				)
-				(justify left)
-			)
-		)
-	)
 	(global_label "Vcc"
 		(shape input)
@@
 			)
 		)
-		(property "Footprint" "Package_SO:SOIC-16_3.9x9.9mm_P1.27mm"
+		(property "Footprint" "Package_DIP:DIP-16_W7.62mm"
 			(at 124.46 104.14 0)
 			(hide yes)
@@
 			)
 		)
-		(property "Footprint" "Package_SO:SOIC-16_3.9x9.9mm_P1.27mm"
+		(property "Footprint" "Package_DIP:DIP-16_W7.62mm"
 			(at 163.83 104.14 0)
 			(hide yes)
@@
 		)
 		(property "Value" "Pin Header 2x8 2,54mm Rounded"
-			(at 270.51 35.56 0)
+			(at 267.97 55.118 0)
 			(show_name no)
 			(do_not_autoplace no)
@@
 		)
 		(property "Footprint" "custom_footprints:PinHeader_2x08_P2.54mm_Vertical"
-			(at 271.526 19.304 0)
-			(show_name no)
-			(do_not_autoplace no)
+			(at 269.748 15.748 0)
+			(show_name no)
+			(do_not_autoplace no)
