File: kicad_alll_smd/4mb mapper nms8280.kicad_sch (KiCad schematic)
At the start: 22 parts, among them IC131 74LS125, IC131B1 74LS125, IC131C1 74LS125, IC147 74LS157, IC147B1 74LS157, IC149 74LS670, IC149B1 74LS670, IC157B1 74LS08, IC180B1 74LS00, J1 Conn_01x10_Pin

Commit message: Publish 4 MB mapper project
Parts:
- IC149, IC149B1: footprint Package_DIP:DIP-16_W7.62mm -> Package_SO:SOIC-16_3.9x9.9mm_P1.27mm
Changed lines of the file:
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@@
 			)
 		)
-		(property "Footprint" "Package_DIP:DIP-16_W7.62mm"
+		(property "Footprint" "Package_SO:SOIC-16_3.9x9.9mm_P1.27mm"
 			(at 124.46 104.14 0)
 			(hide yes)
@@
 			)
 		)
-		(property "Footprint" "Package_DIP:DIP-16_W7.62mm"
+		(property "Footprint" "Package_SO:SOIC-16_3.9x9.9mm_P1.27mm"
 			(at 163.83 104.14 0)
 			(hide yes)
